File: pcb/_autosave-DC_minni.kicad_pcb (KiCad board)
At the start: 4 copper layers, 64 x 85.8 mm, 58 parts, among them J1 DRUCKSENSOR, J2 Encoder, U1 ESP32-DevKitC, U2 USB-C to DIP PCB

Commit message: PCB routing
Parts:
- moved D+1 5.20 mm to (205.3, 88.2)
- moved D-1 1.56 mm to (205.5, 84.3)
- moved REF** 0.93 mm to (201.1, 159.2)
- moved REF** 0.88 mm to (258.0, 158.8)
- renumbered GPIO13 to In, GPIO22 to OUT
Routing:
- net IN: track 0.00 -> 95.6 mm, vias 0 -> 5
- net OUT: track 0.00 -> 83.5 mm, vias 0 -> 1
- net +5V: track 0.00 -> 78.3 mm, vias 0 -> 3
- net ZeroCross: track 0.00 -> 77.0 mm, vias 0 -> 3
- net PWM: track 0.00 -> 69.2 mm, vias 0 -> 3
- net Drucksensor: track 0.40 -> 59.4 mm, vias 0 -> 1
- net +3.3V: track 0.00 -> 44.9 mm, vias 0 -> 3
- net Net-(GPIO23-Pin_1): track 0.00 -> 42.0 mm
- net Net-(GPIO25-Pin_1): track 0.00 -> 38.9 mm, vias 0 -> 3
- net Net-(JSChalter1-Pin_2): track 0.00 -> 35.0 mm, vias 0 -> 4
- net Net-(Detect1-Cathode): track 0.00 -> 22.9 mm
- net Net-(FromMachine1-Pin_1): track 0.00 -> 21.9 mm
- net Net-(GPIO15-Pin_1): track 0.00 -> 17.0 mm, vias 0 -> 1
- net Net-(RSP_01_1-Pad2): track 0.00 -> 16.2 mm, vias 0 -> 2
- net Net-(GPIO2-Pin_1): track 0.00 -> 14.9 mm, vias 0 -> 1
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- added copper zone on B.Cu, net GND
- added copper zone on F.Cu, net GND
