File: pcb/DC_minni.kicad_pcb (KiCad board)
At the start: 4 copper layers, 64 x 85.8 mm, 56 parts, among them J1 DRUCKSENSOR, J2 Encoder, J3 Conn_01x04_Socket, J4 Conn_01x05_Socket, U1 ESP32-DevKitC, U2 USB-C to DIP PCB

Commit message: Updated Pcb again
Routing:
- net IN: track 97.9 -> 96.2 mm
Changed lines of the file:
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@@
-	)
-	(segment
-		(start 216.6 124.271)
-		(end 217.805 125.476)
-		(width 0.4)
-		(layer "F.Cu")
-		(net 3)
 	)
 	(segment
