File: pcb/DC_minni.kicad_sch (KiCad schematic)
At the start: 55 parts, among them J1 DRUCKSENSOR, J2 Encoder, J3 Conn_01x09_Socket, U1 ESP32-DevKitC, U2 USB-C to DIP PCB

Commit message: Updated Pcb again
Parts:
- removed J3: Conn_01x09_Socket, symbol Connector:Conn_01x09_Socket
- added J3: Conn_01x04_Socket, Connector_JST:JST_XH_B4B-XH-A_1x04_P2.50mm_Vertical, symbol Connector:Conn_01x04_Socket
- added J4: Conn_01x05_Socket, Connector_JST:JST_XH_B5B-XH-A_1x05_P2.50mm_Vertical, symbol Connector:Conn_01x05_Socket
Connections:
- net +3.3V: now also J4.3 (Pin_3)
- net Backlight: now also J4.4 (Pin_4)
- net CLK: now also J3.1 (Pin_1)
- net CS: now also J3.4 (Pin_4)
- net DC: now also J4.1 (Pin_1)
- net GND: now also J4.5 (Pin_5)
- net MISO: now also J3.3 (Pin_3)
- net MOSI: now also J3.2 (Pin_2)
- net RST: now also J4.2 (Pin_2)
Changed lines of the file:
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@@
 	(wire
 		(pts
-			(xy 49.53 29.21) (xy 55.88 29.21)
+			(xy 49.53 29.21) (xy 58.42 29.21)
 		)
 		(stroke
@@
 	(wire
 		(pts
-			(xy 49.53 31.75) (xy 55.88 31.75)
+			(xy 49.53 31.75) (xy 58.42 31.75)
 		)
 		(stroke
@@
 	(wire
 		(pts
-			(xy 49.53 36.83) (xy 55.88 36.83)
+			(xy 49.53 36.83) (xy 58.42 36.83)
 		)
 		(stroke
@@
 	(wire
 		(pts
-			(xy 49.53 39.37) (xy 55.88 39.37)
+			(xy 49.53 39.37) (xy 58.42 39.37)
 		)
 		(stroke
@@
 	(wire
 		(pts
-			(xy 49.53 34.29) (xy 55.88 34.29)
+			(xy 49.53 34.29) (xy 58.42 34.29)
 		)
 		(stroke
@@
 	(wire
 		(pts
-			(xy 52.07 49.53) (xy 55.88 49.53)
+			(xy 52.07 49.53) (xy 58.42 49.53)
 		)
 		(stroke
@@
 	(wire
 		(pts
-			(xy 49.53 46.99) (xy 55.88 46.99)
+			(xy 49.53 46.99) (xy 58.42 46.99)
 		)
 		(stroke
@@
 	(wire
 		(pts
-			(xy 49.53 41.91) (xy 55.88 41.91)
+			(xy 49.53 41.91) (xy 58.42 41.91)
 		)
 		(stroke
@@
 	(wire
 		(pts
-			(xy 30.48 44.45) (xy 55.88 44.45)
+			(xy 30.48 44.45) (xy 58.42 44.45)
 		)
 		(stroke
@@
 	)
 	(symbol
+		(lib_id "Connector:Conn_01x05_Socket")
+		(at 63.5 44.45 0)
+		(unit 1)
+		(exclude_from_sim no)
+		(in_bom yes)
+		(on_board yes)
+		(dnp no)
+		(fields_autoplaced yes)
+		(property "Reference" "J4"
+			(at 64.77 43.1799 0)
+			(effects
+				(font
+					(size 1.27 1.27)
+				)
+				(justify left)
+			)
+		)
+		(property "Value" "Conn_01x05_Socket"
+			(at 64.77 45.7199 0)
+			(effects
+				(font
+					(size 1.27 1.27)
+				)
+				(justify left)
+			)
+		)
+		(property "Footprint" "Connector_JST:JST_XH_B5B-XH-A_1x05_P2.50mm_Vertical"
+			(at 63.5 44.45 0)
+			(effects
+				(font
+					(size 1.27 1.27)
+				)
+				(hide yes)
+			)
+		)
+		(property "Datasheet" "~"
+			(at 63.5 44.45 0)
+			(effects
+				(font
+					(size 1.27 1.27)
+				)
+				(hide yes)
+			)
+		)
+		(property "Description" "Generic connector, single row, 01x05, script generated"
+			(at 63.5 44.45 0)
+			(effects
+				(font
+					(size 1.27 1.27)
+				)
+				(hide yes)
+			)
+		)
+		(pin "3"
+		)
+		(pin "1"
+		)
+		(pin "5"
+		)
+		(pin "2"
+		)
+		(pin "4"
+		)
+		(instances
+			(project ""
+				(path "/5c8a4478-a33a-40da-951d-0e2e8bd39df9"
+					(reference "J4")
+					(unit 1)
+				)
+			)
+		)
+	)
+	(symbol
 		(lib_id "mylib:HCPL-817-00AEOPTOKOPPLER")
 		(at 96.52 116.84 0)
@@
 	)
 	(symbol
+		(lib_id "Connector:Conn_01x04_Socket")
+		(at 63.5 31.75 0)
+		(unit 1)
+		(exclude_from_sim no)
+		(in_bom yes)
+		(on_board yes)
+		(dnp no)
+		(fields_autoplaced yes)
+		(property "Reference" "J3"
+			(at 64.77 31.7499 0)
+			(effects
+				(font
+					(size 1.27 1.27)
+				)
+				(justify left)
+			)
+		)
+		(property "Value" "Conn_01x04_Socket"
+			(at 64.77 34.2899 0)
+			(effects
+				(font
+					(size 1.27 1.27)
+				)
+				(justify left)
+			)
+		)
+		(property "Footprint" "Connector_JST:JST_XH_B4B-XH-A_1x04_P2.50mm_Vertical"
+			(at 63.5 31.75 0)
+			(effects
+				(font
+					(size 1.27 1.27)
+				)
+				(hide yes)
+			)
+		)
+		(property "Datasheet" "~"
+			(at 63.5 31.75 0)
+			(effects
+				(font
+					(size 1.27 1.27)
+				)
+				(hide yes)
+			)
+		)
+		(property "Description" "Generic connector, single row, 01x04, script generated"
+			(at 63.5 31.75 0)
+			(effects
+				(font
+					(size 1.27 1.27)
+				)
+				(hide yes)
+			)
+		)
+		(pin "2"
+		)
+		(pin "4"
+		)
+		(pin "3"
+		)
+		(pin "1"
+		)
+		(instances
+			(project ""
+				(path "/5c8a4478-a33a-40da-951d-0e2e8bd39df9"
+					(reference "J3")
+					(unit 1)
+				)
+			)
+		)
+	)
+	(symbol
 		(lib_id "power:+3.3V")
 		(at 52.07 96.52 90)
@@
 					(unit 1)
 				)
-			)
-		)
-	)
-	(symbol
-		(lib_id "Connector:Conn_01x09_Socket")
-		(at 60.96 39.37 0)
-		(unit 1)
-		(exclude_from_sim no)
-		(in_bom yes)
-		(on_board yes)
-		(dnp no)
-		(fields_autoplaced yes)
-		(property "Reference" "J3"
-			(at 62.23 38.0999 0)
-			(effects
-				(font
-					(size 1.27 1.27)
-				)
-				(justify left)
-			)
-		)
-		(property "Value" "Conn_01x09_Socket"
-			(at 62.23 40.6399 0)
-			(effects
-				(font
-					(size 1.27 1.27)
-				)
-				(justify left)
-			)
-		)
-		(property "Footprint" ""
-			(at 60.96 39.37 0)
-			(effects
-				(font
-					(size 1.27 1.27)
-				)
-				(hide yes)
-			)
-		)
-		(property "Datasheet" "~"
-			(at 60.96 39.37 0)
-			(effects
-				(font
-					(size 1.27 1.27)
-				)
-				(hide yes)
-			)
-		)
-		(property "Description" "Generic connector, single row, 01x09, script generated"
-			(at 60.96 39.37 0)
-			(effects
-				(font
-					(size 1.27 1.27)
-				)
-				(hide yes)
-			)
-		)
-		(pin "6"
-		)
-		(pin "8"
-		)
-		(pin "1"
-		)
-		(pin "5"
-		)
-		(pin "4"
-		)
-		(pin "7"
-		)
-		(pin "9"
-		)
-		(pin "3"
-		)
-		(pin "2"
-		)
-		(instances
-			(project ""
-				(path "/5c8a4478-a33a-40da-951d-0e2e8bd39df9"
-					(reference "J3")
-					(unit 1)
-				)

Commit message: update pressure pin
Changed lines of the file:
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@@
 (kicad_sch
-	(version 20231120)
+	(version 20250114)
 	(generator "eeschema")
-	(generator_version "8.0")
+	(generator_version "9.0")
 	(paper "A4")
 	(junction
@@
 		)
 	)
+	(embedded_fonts no)
 )
